Commit message: Ready for evaluation.

File: sweeping_robot/urdf/sweeping_robot.xacro (robot description, xacro)
@@ -12,7 +12,7 @@
   </joint>
   <link name="chassis">
-    <pose>0 0 0.16 0 0 0</pose>
-    <inertial>
-      <mass value="15.0"/>
+    <pose>0 0 0.15 0 0 0</pose>
+    <inertial>
+      <mass value="10.0"/>
       <origin xyz="0.0 0 0" rpy="0 0 0"/>
       <inertia
@@ -34,8 +34,54 @@
       </geometry>
     </visual>
+    <!-- front caster -->
+    <collision name='front_caster_collision'>
+      <origin xyz="0.10 0 -0.05" rpy=" 0 0 0"/>
+      <geometry>
+        <sphere radius="0.10"/>
+      </geometry>
+      <surface>
+        <friction>
+          <ode>
+            <mu>0</mu>
+            <mu2>0</mu2>
+            <slip1>1.0</slip1>
+            <slip2>1.0</slip2>
+          </ode>
+        </friction>
+      </surface>
+    </collision>
+    <visual name='front_caster_visual'>
+      <origin xyz="0.10 0 -0.05" rpy=" 0 0 0"/>
+      <geometry>
+        <sphere radius="0.10"/>
+      </geometry>
+    </visual>
+    <!-- back caster -->
+    <collision name='back_caster_collision'>
+      <origin xyz="-0.10 0 -0.05" rpy=" 0 0 0"/>
+      <geometry>
+        <sphere radius="0.10"/>
+      </geometry>
+      <surface>
+        <friction>
+          <ode>
+            <mu>0</mu>
+            <mu2>0</mu2>
+            <slip1>1.0</slip1>
+            <slip2>1.0</slip2>
+          </ode>
+        </friction>
+      </surface>
+    </collision>
+    <visual name='back_caster_visual'>
+      <origin xyz="-0.10 0 -0.05" rpy=" 0 0 0"/>
+      <geometry>
+        <sphere radius="0.10"/>
+      </geometry>
+    </visual>
   </link>
   <!-- left wheel -->
   <joint type="continuous" name="left_wheel_hinge">
-    <origin xyz="+0.12 +0.12 -0.11" rpy="0 0 0"/>
+    <origin xyz="+0.00 +0.15 -0.10" rpy="0 0 0"/>
     <parent link="chassis"/>
     <child link="left_wheel"/>
@@ -46,5 +92,5 @@
   <link name="left_wheel">
     <inertial>
-      <mass value="3.0"/>
+      <mass value="1.0"/>
       <origin xyz="0.0 0 0" rpy=" 0 1.5707 1.5707"/>
       <inertia
@@ -69,5 +115,5 @@
   <!-- right wheel -->
   <joint type="continuous" name="right_wheel_hinge">
-    <origin xyz="+0.12 -0.12 -0.11" rpy="0 0 0"/>
+    <origin xyz="+0.00 -0.15 -0.10" rpy="0 0 0"/>
     <parent link="chassis"/>
     <child link="right_wheel"/>
@@ -78,5 +124,5 @@
   <link name="right_wheel">
     <inertial>
-      <mass value="3.0"/>
+      <mass value="1.0"/>
       <origin xyz="0.0 0 0" rpy=" 0 1.5707 1.5707"/>
       <inertia
@@ -99,36 +145,4 @@
     </visual>
   </link>
-  <!-- back wheel -->
-  <joint type="continuous" name="back_wheel_hinge">
-    <origin xyz="-0.15 0.0 -0.11" rpy="0 0 0"/>
-    <parent link="chassis"/>
-    <child link="back_wheel"/>
-    <axis xyz="0 1 0" rpy="0 0 0"/>
-    <limit effort="10000" velocity="1000"/>
-    <dynamics damping="1.0" friction="1.0"/>
-  </joint>
-  <link name="back_wheel">
-    <inertial>
-      <mass value="3.0"/>
-      <origin xyz="0.0 0 0" rpy=" 0 1.5707 1.5707"/>
-      <inertia
-          ixx="0.1" ixy="0" ixz="0"
-          iyy="0.1" iyz="0"
-          izz="0.1"
-      />
-    </inertial>
-    <collision name="back_wheel_collision">
-      <origin xyz="0 0 0" rpy=" 0 1.5707 1.5707"/>
-      <geometry>
-        <cylinder length="0.02" radius="0.05"/>
-      </geometry>
-    </collision>
-    <visual name="back_wheel_visual">
-      <origin xyz="0 0 0" rpy=" 0 1.5707 1.5707"/>
-      <geometry>
-        <cylinder length="0.02" radius="0.05"/>
-      </geometry>
-    </visual>
-  </link>
   <!-- RGB-D camera -->
   <joint type="fixed" name="rgbd_camera_joint">
